File: KiCAD_files/PowerLeg2.kicad_sch (KiCad schematic)
At the start: 51 parts

Commit message: Added feeder project alpha version
Former-commit-id: 38773bad2925cccbdf57e9531d71dd427b0662b4
Parts:
- removed C? (x2): 100nF, Capacitor_SMD:C_0805_2012Metric, symbol Device:C_Small
- removed J? (x4): Conn_01x01, Footprints:0906_millmax, symbol Connector_Generic:Conn_01x01
- added C302, C304, C309, C314, C315, C316, C320: 100nF, Capacitor_SMD:C_0805_2012Metric, symbol Device:C_Small
- added C305, C306: 33pF, Capacitor_SMD:C_0805_2012Metric, symbol Device:C_Small
- added C313, C319: 20pF, Capacitor_SMD:C_0805_2012Metric, symbol Device:C_Small
- added C317: 10uF, Capacitor_SMD:C_1210_3225Metric, symbol Device:C_Small
- added C318: 1uF, Capacitor_SMD:C_0805_2012Metric, symbol Device:C_Small
- added D301: STTH4R02U, Diode_SMD:D_SMB, symbol Device:D_Schottky
- added J301, J302, J303, J304: Conn_01x01, Footprints:0906_millmax, symbol Connector_Generic:Conn_01x01
- added R301, R302, R320: 51, Resistor_SMD:R_0805_2012Metric, symbol Device:R
- added R303: 20k, Resistor_SMD:R_0805_2012Metric, symbol Device:R
- added R307: 2.2, Resistor_SMD:R_0805_2012Metric, symbol Device:R
- added R309, R321: 1k, Resistor_SMD:R_0805_2012Metric, symbol Device:R_Small
- added R322: 1k, Resistor_SMD:R_0805_2012Metric, symbol Device:R
- added U303: UCC21222DR, Package_SO:SOIC-16W_7.5x10.3mm_P1.27mm, symbol Driver_FET:UCC21520DW
- added U306: SFH617A-2X009T, Package_DIP:SMDIP-4_W7.62mm, symbol Isolator:SFH617A-2X009T
- R316: renamed from R?; value 200k -> 62k
- R317: renamed from R?; value 200k -> 43k
- R318: renamed from R?; value 82k -> 43k
- R319: renamed from R?; value 82k -> 62k
- gave numbers to parts that had none: 41
Connections:
- net +5VD: now also C302.1, C304.1, R309.1, R321.1, U303.3 (VCCI), U303.8 (VCCI)
- net DGND: now also C314.2, C320.2; no longer R317.1
- net GNDREF: now also C315.2, C317.2, R322.1, U303.9 (VSSB); no longer J308.1 (Pin_1)
- net IILow2_op: now also C319.2
- net PWM_H2: now also U303.15 (OUTA)
- net PWM_L2: now also U303.10 (OUTB)
- net SW_Node2: now also C316.2, C318.2, U303.14 (VSSA)
- net VILow2_op: now also C313.2
- net Vref: now also R317.1
- net at R317.2, R319.1, U305.3 (-): now also C319.1
- net at R305.2, R308.1, U304.3 (-): now also C313.1
- net Neutral_GND_cmd renamed +12V
- net +12V: now also C315.1, C317.1, R307.2, U303.11 (VDDB), U306.4; no longer J307.1 (Pin_1)
- new net: D301.2 (A), R307.1
- new net: C305.2, R301.2, U303.1 (INA)
- new net: R320.2, U306.2
- new net: C306.1, R302.2, U303.2 (INB)
- new net: C316.1, C318.1, D301.1 (K), U303.16 (VDDA)
- new net: C309.1, R303.2, U303.6 (DT)
- new net: R322.2, U306.3
- new net GNDD: C302.2, C304.2, C305.1, C306.2, C309.2, J303.1 (Pin_1), J304.1 (Pin_1), J308.1 (Pin_1), R303.1, R320.1, U303.4 (GND), U303.5 (DIS)
- new net HRTIM1_CHA1: J301.1 (Pin_1), R301.1
- new net HRTIM1_CHA2: J302.1 (Pin_1), R302.1
- new net N_GND: J307.1 (Pin_1), U306.1
- new net U13_5V: C314.1, C320.1, R309.2, R321.2
Other:
- moved on the sheet: C301, C303, C307, C308, C310, C311, C312, C321, C322, C323, Cs301, D302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
