File: KiCAD_files/_autosave-Power.kicad_pcb (KiCad board)
At the start: 4 copper layers, 100 x 100 mm, 206 parts, among them J1 Conn_01x01, J10 Conn_01x01, J101 2604-1102, J102 2604-1102, J103 2604-1102, J104 Conn_01x01, J105 Conn_01x01, J106 Conn_01x01, J107 Conn_01x01, J108 Conn_01x01, J109 Conn_01x01, J110 Conn_01x01, J111 Conn_01x01, J112 Conn_01x01, J113 Conn_01x01, J114 Conn_01x01, J115 Conn_01x01, J116 Conn_01x01, J117 2604-1102, J118 2604-1102, J2 Conn_01x01, J201 Conn_01x01, J202 Conn_01x01, J203 Conn_01x01, J204 Conn_01x01, J205 Conn_01x01, J206 Conn_01x01, J207 Conn_01x01, J208 Conn_01x01, J209 Conn_01x01, J210 Conn_01x01, J3 Conn_01x01, J4 Conn_01x01, J5 Conn_01x01, J6 Conn_01x01, J7 Conn_01x01, J8 Conn_01x01, J9 Conn_01x01, Q1 IPD200N15N3, Q2 IPD200N15N3, Q201 IPD200N15N3, Q202 IPD200N15N3, Q203 IPD200N15N3, Q3 IPD200N15N3, U1 AMC1100DUB, U101 AMC1311, U102 OPA316, U103 OPA316, U104 +-20A, U2 ACS730xLCTR-20AB, U201 AMC1100DUB, U202 ACS730xLCTR-20AB, U203 UCC21222DR, U204 OPA316, U205 OPA316, U206 SFH617A-2X009T, U3 UCC21222DR, U4 OPA316, U5 OPA316, U6 SFH617A-2X009T

Commit message: WIP routing the power board
Former-commit-id: fec71ccccc2062c429ca6048755d91568543f1a5
Parts:
- moved R7 16.5 mm to (69.0, 110.7)
- moved U104 12.3 mm to (55.0, 120.8), turned to 90 degrees
- moved C120 11.9 mm to (49.2, 117.6), turned to -90 degrees
- moved R24 9.97 mm to (51.2, 117.7), turned to -90 degrees
- moved R110 9.08 mm to (50.4, 108.2), turned to -90 degrees
- moved C118 9.07 mm to (58.8, 117.6), turned to 90 degrees
- moved J116 8.50 mm to (57.4, 106.4), turned to 90 degrees
- moved J115 8.12 mm to (54.8, 106.4), turned to 90 degrees
- moved R11 7.44 mm to (82.3, 102.6)
- moved D3 7.44 mm to (83.0, 104.8)
- moved C119 6.99 mm to (52.4, 108.2), turned to 90 degrees
- moved D2 6.70 mm to (78.2, 104.8)
- moved R10 6.70 mm to (78.8, 102.6)
- moved C16 6.50 mm to (86.6, 109.8), turned to -90 degrees
- moved C117 6.42 mm to (59.6, 110.2), turned to 90 degrees
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Routing:
- net DGND: track 24.4 -> 65.6 mm, vias 1 -> 12
- net /Power Leg 2/SW_Node: track 0.00 -> 36.7 mm, vias 0 -> 2
- net GNDREF: track 34.1 -> 68.2 mm, vias 16 -> 25
- net +12V: track 45.3 -> 79.3 mm, vias 3 -> 5
- net NGND: track 0.00 -> 18.3 mm, vias 1 -> 16
- net Net-(D3-Pad2): track 0.00 -> 15.2 mm, vias 0 -> 2
- net Net-(D2-Pad2): track 0.00 -> 15.0 mm, vias 0 -> 2
- net /Power Leg 2/PWM_H1: track 0.00 -> 9.33 mm
- net /Power Leg 2/PWM_L1: track 0.00 -> 9.30 mm
- net /Power Leg 1/IILow1_op: track 0.00 -> 9.04 mm
- net /Power Leg 2/IILow1_op: track 0.00 -> 9.04 mm
- net /Power Leg 1/IILow1: track 0.00 -> 7.87 mm
- net /Power Leg 2/IILow1: track 0.00 -> 7.87 mm
- net Net-(C15-Pad1): track 0.00 -> 7.64 mm
- net Net-(C13-Pad1): track 0.00 -> 7.08 mm
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- added copper zone on F.Cu, net /Power Leg 2/SW_Node
- added copper zone on F.Cu, net /V2_Low
- added copper zone on In1.Cu, net DGND
- added copper zone on F.Cu, net NGND
- added copper zone on F.Cu, net Net-(L1-Pad1)
