File: KiCAD_files/Microcontroller.kicad_pcb (KiCad board)
At the start: 4 copper layers, 100 x 100 mm, 132 parts, among them J1 Conn_01x02, J2 RJ45_LED_Shielded, J3 RJ45_LED_Shielded, J4 Conn_01x06_Male, J5 Conn_01x06_Male, J6 Conn_01x02, J7 Power, J8 Conn_02x07_Odd_Even, J9 Conn_01x03, SW1 SW_Push, U1 STM32G474RE, U10 MCP1799T-5002H/TT, U2 AT25xxx, U3 TCAN334GDR, U4 AP1117-33, U5 UCC21222DR, U6 UCC21222DR, U7 SFH617A-2X009T, U8 RFM-0505s, U9 CME0512S3C, Y1 ECS-240-10-33-AGM-TR - 24MHz

Commit message: Created a first routed STM32G4 module and ordered it in JLCPCB
Former-commit-id: 49804de64bb80eadc7f05c9bfca13c93680f06aa
Other:
- net class Default removed

Commit message: WIP: mooving to a single board implementation with 160x100 form factor.
Former-commit-id: e8c19d5fc5237412fb5a003591d44756dbc6e173
Parts:
- removed C1, C10, C11, C13, C20, C21, C22, C25, C26, C30, C31, C32, C42, C5, C7, C8, C9: 100nF, Capacitor_SMD:C_0805_2012Metric
- removed C12, C41: 1µF, Capacitor_SMD:C_0805_2012Metric
- removed C14: 10nF, Capacitor_SMD:C_0805_2012Metric
- removed C15, C16: 47uF, Capacitor_SMD:CP_Elec_6.3x7.7
- removed C17, C18, C27, C28: 33pF, Capacitor_SMD:C_0805_2012Metric
- removed C19, C24, C34, C39, C40: 10uF, Capacitor_SMD:C_1210_3225Metric
- removed C23, C33: 1uF, Capacitor_SMD:C_0805_2012Metric
- removed C29: 10uF, Capacitor_SMD:CP_Elec_8x11.9
- removed C3, C4: 12pF, Capacitor_SMD:C_0805_2012Metric
- removed C6: 4,7uF, Capacitor_SMD:C_0805_2012Metric
- removed D10, D11: STTH4R02U, Diode_SMD:D_SMB
- removed D3, D4, D5, D6, D7, D8, D9: 3.3V, Diode_SMD:D_SOD-123
- removed FB1: 100Ohm @ 100MHz, Resistor_SMD:R_0805_2012Metric
- removed J1, J6: Conn_01x02, Footprints:PTSM-0,5-2-HH0-SMD
- removed J7: Power, Footprints:3D_Footprint_Power
- removed J8: Conn_02x07_Odd_Even, Connector_PinHeader_1.27mm:PinHeader_2x07_P1.27mm_Vertical_SMD
- removed J9: Conn_01x03, Connector_PinHeader_2.54mm:PinHeader_1x03_P2.54mm_Vertical
- removed LED1: LED, LED_SMD:LED_0805_2012Metric
- removed LED2: PWR, LED_SMD:LED_0805_2012Metric
- removed PS5: VXO78xxx, Footprints:CONV_VXO78012-500-M
- removed R14, R17, R18, R21, R9: 51, Resistor_SMD:R_0805_2012Metric
- removed R15, R19: 20k, Resistor_SMD:R_0805_2012Metric
- removed R16, R20: 2.2, Resistor_SMD:R_0805_2012Metric
- removed R2, R24, R3, R4, R5, R6, R7, R8: 100, Resistor_SMD:R_0805_2012Metric
- removed R22: 1k, Resistor_SMD:R_0805_2012Metric
- removed R23: 220, Resistor_SMD:R_0805_2012Metric
- removed R26, R28: 330, Resistor_SMD:R_0805_2012Metric
- removed SW1: SW_Push, Button_Switch_SMD:SW_Push_1P1T_NO_CK_KMR2
- removed SWD1: Conn_01x06_Female, Connector_PinHeader_2.54mm:PinHeader_1x06_P2.54mm_Vertical
- removed TP1, TP12, TP2, TP3, TP4, TP5, TP6, TP7, TP8: TestPoint, TestPoint:TestPoint_THTPad_D2.0mm_Drill1.0mm
- removed U2: AT25xxx, Footprints:SOIC-8_3.9x4.9mm_P1.27mm
- removed U4: AP1117-33, Package_TO_SOT_SMD:SOT-223-3_TabPin2
- removed U5, U6: UCC21222DR, Footprints:SOIC-16_3.9x9.9mm_P1.27mm
- removed U7: SFH617A-2X009T, Package_DIP:SMDIP-4_W7.62mm
- removed Y1: ECS-240-10-33-AGM-TR - 24MHz, Crystal:Crystal_SMD_3225-4Pin_3.2x2.5mm
- added JP5: Jumper, Connector_PinHeader_2.54mm:PinHeader_1x02_P2.54mm_Vertical, F.Cu at (58.6, 172.9)
- added P1: Power2, Footprints:3D_Footprint_PowerV1.1.3, F.Cu at (57.0, 70.0)
- JP1: footprint Jumper:SolderJumper-2_P1.3mm_Open_Pad1.0x1.5mm -> Connector_PinHeader_2.54mm:PinHeader_1x02_P2.54mm_Vertical
- PS4: value PQDE6W-Q110-S5-D -> Feeder; footprint Footprints:PQDE6W-Q110-S5-D -> Footprints:Feeder
- TH1: moved to F.Cu
- U1: value STM32G474RE -> OwnTech; footprint Package_QFP:LQFP-64_10x10mm_P0.5mm -> Footprints:OwnTech_MCU
- U9: footprint Converter_DCDC:Converter_DCDC_muRata_CRE1xxxxxx3C_THT -> Converter_DCDC:Converter_DCDC_Murata_CRE1xxxxxx3C_THT
- moved JP4 145.9 mm to (-31.0, 41.0), turned to 180 degrees
- moved TH1 114.8 mm to (44.1, 58.8), turned to 0 degrees
- moved J5 107.8 mm to (-25.0, 47.8)
- moved BT1 104.6 mm to (210.6, 56.0), turned to 180 degrees
- moved C36 104.4 mm to (18.8, 113.1), turned to 90 degrees
- moved C38 103.4 mm to (18.8, 107.5), turned to 90 degrees
- moved U10 97.5 mm to (18.0, 119.0), turned to 180 degrees
- moved C2 97.0 mm to (119.1, 24.8), turned to 0 degrees
- moved U9 96.3 mm to (22.4, 106.5), turned to 0 degrees
- moved C43 96.2 mm to (18.6, 123.4), turned to 90 degrees
- moved JP2 95.2 mm to (198.8, 51.2), turned to 180 degrees
- moved C44 91.6 mm to (21.1, 123.6), turned to 90 degrees
- moved U3 88.2 mm to (119.1, 29.8), turned to -90 degrees
- moved JP3 84.5 mm to (166.7, 78.5)
- moved TP14 82.7 mm to (112.3, 29.6), turned to 180 degrees
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Connections:
- net +5P renamed +5VP
- net +5V renamed +5VN
- net /N renamed NGND
- net GNDREF renamed GND
- net Net-(U1-Pad2) renamed HRTIM_CHC1
- net Net-(U1-Pad35) renamed V_{I1Low}
- net Net-(U1-Pad36) renamed I_{I1Low}
- net Net-(U1-Pad4) renamed HRTIM_CHC2
- BT1 pad 2: GNDD -> DGND
- C2 pad 2: GNDD -> DGND
- C37 pad 2: GNDD -> DGND
- C38 pad 2: GNDD -> DGND
- D2 pad 1: GNDD -> DGND
- J2 pad 6: Net-(J2-Pad6) -> unconnected-(J2-Pad6)
- J2 pad 8: Net-(J2-Pad8) -> unconnected-(J2-Pad8)
- J2 pad SH: GNDD -> unconnected-(J2-PadSH)
- J3 pad 6: Net-(J3-Pad6) -> unconnected-(J3-Pad6)
- J3 pad 8: Net-(J3-Pad8) -> unconnected-(J3-Pad8)
- J3 pad SH: GNDD -> unconnected-(J3-PadSH)
- J4 pad 3: /USART1_RX -> USART1_{RX}
- J4 pad 4: /USART1_TX -> USART1_{TX}
- J4 pad 5: GNDD -> DGND
- J5 pad 1: GNDD -> DGND
- J5 pad 3: /SPI3_MISO -> SPI3_{MISO}
- J5 pad 4: /SPI3_MOSI -> SPI3_{MOSI}
- JP3 pad 1: /DAC2 -> DAC2
- JP3 pad 2: /VREF1024 -> VREF1024
- PS4 pad 1: (no net) -> V_{IHighpower}
- PS4 pad 3: /VI_high -> DGND
- R25 pad 1: /Temp -> Temp
- TH1 pad 1: /Temp -> Temp
- TH1 pad 2: GNDD -> DGND
- TP13 pad 1: /FDCAN1_TX -> FDCAN1_{TX}
- TP14 pad 1: /FDCAN1_RX -> FDCAN1_{RX}
- U1 pad 1: +BATT -> unconnected-(U1-Pad1)
- U1 pad 10: /I_high_mcu -> unconnected-(U1-Pad10)
- U1 pad 11: /V_high_mcu -> unconnected-(U1-Pad11)
- U1 pad 12: /V1_low_mcu -> HRTIM_CHA2
- U1 pad 13: /I1_low_mcu -> DGND
- U1 pad 14: /STLINK_RX -> HRTIM_CHA1
- U1 pad 15: GNDD -> unconnected-(U1-Pad15)
- U1 pad 16: +3V3 -> unconnected-(U1-Pad16)
- U1 pad 17: /STLINK_TX -> unconnected-(U1-Pad17)
- U1 pad 18: /SPI3_CS -> DGND
- U1 pad 19: /LED_BUILTIN -> unconnected-(U1-Pad19)
- U1 pad 20: /DAC2 -> SPI3_{MISO}
- U1 pad 21: /EEPROM_WP -> SPI3_{MOSI}
- U1 pad 22: /SPI3_CS2 -> DGND
- U1 pad 23: Net-(U1-Pad23) -> USART1_{TX}
- U1 pad 24: /EEPROM_HOLD -> USART1_{RX}
- U1 pad 25: /Temp_mcu -> DGND
- U1 pad 26: Net-(U1-Pad26) -> FDCAN1_{RX}
- U1 pad 27: GNDD -> FDCAN1_{TX}
- U1 pad 28: /VREF2048 -> unconnected-(U1-Pad28)
- U1 pad 29: +3.3VA -> DGND
- U1 pad 3: Net-(U1-Pad3) -> DGND
- U1 pad 30: /CAN1_STB -> V_{I2Low}
- U1 pad 31: GNDD -> I_{I2Low}
- U1 pad 32: +3V3 -> I_{IHigh}
- U1 pad 33: /N_GND -> V_{IHigh}
- U1 pad 34: Net-(U1-Pad34) -> DGND
- U1 pad 37: Net-(U1-Pad37) -> BOOT
- U1 pad 38: Net-(U1-Pad38) -> unconnected-(U1-Pad38)
- U1 pad 39: Net-(U1-Pad39) -> DGND
- U1 pad 40: Net-(U1-Pad40) -> DAC2
- U1 pad 41: Net-(U1-Pad41) -> unconnected-(U1-Pad41)
- U1 pad 42: /HRTIM1_CHA1 -> +3V3
- U1 pad 43: /HRTIM1_CHA2 -> Temp
- U1 pad 44: /HRTIM1_CHB1 -> DGND
- U1 pad 45: /HRTIM1_CHB2 -> +BATT
- U1 pad 46: /HRTIM1_FLT1 -> +5VD
- U1 pad 5: /HSE_IN -> unconnected-(U1-Pad5)
- U1 pad 6: /HSE_OUT -> unconnected-(U1-Pad6)
- U1 pad 7: /NRST -> unconnected-(U1-Pad7)
- U1 pad 8: /V2_low_mcu -> DGND
- U1 pad 9: /I2_low_mcu -> unconnected-(U1-Pad9)
- U3 pad 1: /FDCAN1_TX -> FDCAN1_{TX}
- U3 pad 2: GNDD -> DGND
- U3 pad 4: /FDCAN1_RX -> FDCAN1_{RX}
- U3 pad 5: Net-(U3-Pad5) -> unconnected-(U3-Pad5)
- U8 pad 1: GNDD -> DGND
- U9 pad 1: GNDD -> DGND
Routing:
- net GNDD: track 160.0 -> 0.00 mm, vias 57 -> 0
- net +5VD: track 108.8 -> 2.72 mm, vias 7 -> 0
- net GND: track 104.6 -> 0.00 mm, vias 23 -> 0
- net /GND_CAN: track 85.4 -> 0.00 mm, vias 3 -> 0
- net /CAN1_STB: track 85.1 -> 0.00 mm, vias 4 -> 0
- net /SPI3_SCK: track 80.4 -> 0.08 mm, vias 2 -> 0
- net /SWO: track 75.4 -> 0.00 mm, vias 2 -> 0
- net /CAN_L: track 73.9 -> 0.00 mm
- net /SWDIO: track 73.5 -> 0.00 mm, vias 2 -> 0
- net /SPI3_MOSI: track 72.4 -> 0.00 mm, vias 3 -> 0
- net /SPI3_MISO: track 71.0 -> 0.00 mm, vias 3 -> 0
- net /CAN_H: track 69.0 -> 0.00 mm
- net +3V3: track 65.5 -> 0.00 mm, vias 11 -> 0
- net /SWCLK: track 59.1 -> 0.00 mm, vias 2 -> 0
- net /USART1_RX: track 55.0 -> 0.00 mm, vias 2 -> 0
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- removed copper zone on In2.Cu, net +12V
- removed copper zone on F.Cu, net +3V3
- removed copper zone on In2.Cu, net +3V3
- removed copper zone on F.Cu, net +5VD
- removed copper zone on In2.Cu, net +5VD
- removed copper zone on In2.Cu, net /+12VD
- removed copper zone on F.Cu, net GND
- removed copper zone on In1.Cu, net GND
- removed copper zone on F.Cu, net GNDD
- removed copper zone on In1.Cu, net GNDD
Other:
- outline, holes or cut-outs redrawn
- board text added: "V1.1.3"
- board text removed: "2.048V"
- board text removed: "PWMH1"
- board text removed: "PWMH2"
- board text removed: "PWML1"
- board text removed: "PWML2"
- board text removed: "RST"
- board text removed: "STDC14"
- board text removed: "V1.1.2"
- board text removed: "VBAT"
