File: KiCAD_files/PowerLeg1.kicad_sch (KiCad schematic)
At the start: 78 parts, among them Q201 IPD200N15N3, Q202 IPD200N15N3, Q203 IPD200N15N3, U201 AMC1100DUB, U202 ACS730xLCTR-20AB, U203 UCC21222DR, U204 OPA316, U205 OPA316, U206 HMHA2801A, U207 HMHA2801A

Commit message: Feature Freeze PCB ordered
Former-commit-id: 656e77d39b103ec58b17965582500bfb0a5b80a0
Parts:
- TP310: renamed from TP210; footprint Footprints:TestPoint_THTPad_D1.5mm_Drill0.7mm -> TestPoint:TestPoint_Pad_D1.0mm
- TP311: renamed from TP211; footprint Footprints:TestPoint_THTPad_D1.5mm_Drill0.7mm -> TestPoint:TestPoint_Pad_D1.0mm
- TP312: renamed from TP212; footprint Footprints:TestPoint_THTPad_D1.5mm_Drill0.7mm -> TestPoint:TestPoint_Pad_D1.0mm
- TP313: renamed from TP213; footprint Footprints:TestPoint_THTPad_D1.5mm_Drill0.7mm -> TestPoint:TestPoint_Pad_D1.0mm
- renumbered C201 to C301, C202 to C302, C203 to C303, C204 to C304, C205 to C305, C206 to C306, C207 to C307, C208 to C308, C209 to C309, C210 to C310, C211 to C311, C212 to C312, C213 to C313, C214 to C314, C215 to C315, C216 to C316, C217 to C317, C218 to C318, C219 to C319, C220 to C320, C221 to C321, C222 to C322, C223 to C323, D201 to D301, D202 to D302, D203 to D303, D204 to D304, D205 to D305, L201 to L301, Q201 to Q301, Q202 to Q302, Q203 to Q303, R201 to R301, R202 to R302, R203 to R303, R204 to R304, R205 to R305, R206 to R306, R207 to R307, R208 to R308, R209 to R309, R210 to R310, R211 to R311, R212 to R312, R213 to R313, R214 to R314, R215 to R315, R216 to R316, R217 to R317, R218 to R318, R219 to R319, R220 to R320, R221 to R321, R222 to R322, R223 to R323, R224 to R324, R225 to R325, R226 to R326, TP201 to TP301, TP202 to TP302, TP203 to TP303, TP204 to TP304, TP205 to TP305, TP206 to TP306, TP207 to TP307, TP208 to TP308, TP209 to TP309, U201 to U301, U202 to U302, U203 to U303, U204 to U304, U205 to U305, U206 to U306, U207 to U307

Commit message: Added necessary information for BOM ordering
Former-commit-id: 116c703b052ef693f4f6c94bbef521d6efde9abc
Parts:
- C301, C304, C314: #manf (none) -> C1206C104K5RAC7867; Manf# (none) -> C1206C104K5RAC7867
- C302, C305, C311, C316, C317: Manf# CC0805KRX7R9BB104 -> C0805C104K5RACTU
- C303: Manf# (none) -> EEE-FN2A470UL
- C306, C309, C312: Manf# (none) -> 12101C475K4T2A
- C307, C308: value 33pF -> 20pF; Manf# C0805C330J5GACTU -> CC0805JRNPO9BN200
- C310: #manf (none) -> CL21C102JCFNNNE; Manf# (none) -> CL21C102JCFNNNE
- C313, C320: Manf# (none) -> C0805C104K5RACTU
- C315, C321: Manf# (none) -> CC0805JRNPO9BN200
- C318: #manf (none) -> 12105C106KAT2A; Manf# CL32B106KBJZW6E -> 12105C106KAT2A
- C319: #manf (none) -> UMK212B7105KGHT; Manf# CL21B105KBFNFNE -> UMK212B7105KGHT
- C322: value 100nF -> 1nF 200V; Manf# (none) -> CL21B103KDCNNNC
- C323: #manf (none) -> C1210C104M2RACTU; Manf# (none) -> C1210C104M2RACTU
- D301: Manf# STTH4R02U -> PU3DBH
- D302, D303: value STPS0520Z -> PMEG2010AEJ,115; Manf# (none) -> PMEG2010AEJ,115
- D304, D305: value STTH1002CB -> S115FA; Manf# (none) -> S115FA
- L301: Manf# (none) -> SRP1510CA-330M
- Q301, Q302, Q303: Manf# (none) -> IPD200N15N3
- R301, R306, R311, R312, R319, R320, R321: Manf# (none) -> CR0805-FX-1001ELF
- R302: value 150K -> 150k; Manf# (none) -> CR0805-FX-1503ELF
- R303: value 470 -> 470R; Manf# (none) -> CR0805-FX-4700ELF
- R304, R305, R324, R326: value 51 -> 51R; Manf# RT0805FRE0751RL -> CR0805-FX-51R0ELF
- R307: Manf# PCF-W0805LF-03-2002-B-P-LT -> CR0805-FX-2002ELF
- R308, R309: Manf# (none) -> CR0805-FX-2702ELF
- R310, R313: Manf# (none) -> CR0805-FX-1202ELF
- R314: value 2.2 -> 2.2R
- R315, R316: value 2,2 -> 2.2R; Manf# (none) -> CR0805AF/-2R20EAS
- R317, R323: Manf# (none) -> CR0805-FX-5901ELF
- R318, R322: Manf# (none) -> CR0805-FX-2002ELF
- R325: Manf# RC0805FR-071KL -> CR0805-FX-1001ELF
- TP301, TP302, TP303, TP304, TP305, TP306, TP307, TP308, TP309, TP310, TP311, TP312, TP313: DNP (none) -> x
- U301: Manf# (none) -> AMC1100DUB
- U302: Manf# (none) -> ACS730xLCTR-20AB
- U304, U305: Manf# (none) -> MCP6486UT-E/LT
- U306, U307: #manf (none) -> HMHA2801A; Manf# SFH617A-2X009T -> HMHA2801A

Commit message: modified components references
Former-commit-id: 78eae5a79aa085afeb122b22fc422d089bf318c8
Parts:
- U306, U307: Manf# HMHA2801A -> FODM217A
Changed lines of the file:
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@@
       (effects (font (size 1.27 1.27)) hide)
     )
-    (property "Manf#" "HMHA2801A" (id 4) (at 107.95 123.19 0)
+    (property "Manf#" "FODM217A" (id 4) (at 107.95 123.19 0)
       (effects (font (size 1.27 1.27)) hide)
     )
@@
       (effects (font (size 1.27 1.27)) hide)
     )
-    (property "Manf#" "HMHA2801A" (id 4) (at 234.95 143.51 0)
-      (effects (font (size 1.27 1.27)) hide)
-    )
+    (property "Manf#" "FODM217A" (id 4) (at 234.95 143.51 0)
+      (effects (font (size 1.27 1.27)) hide)
+    )

Commit message: Push up-to-date design files
Former-commit-id: f8cc17d9887a3e68c026953a0d17b74481171696
Parts:
- C201: renamed from C301; DNP (none) -> x
- C202: renamed from C302; DNP (none) -> x
- C203: renamed from C303; DNP (none) -> x
- C204: renamed from C304; DNP (none) -> x
- C205: renamed from C305; DNP (none) -> x
- C206: renamed from C306; DNP (none) -> x
- C207: renamed from C307; DNP (none) -> x
- C208: renamed from C308; DNP (none) -> x
- C209: renamed from C309; DNP (none) -> x
- C210: renamed from C310; DNP (none) -> x
- C211: renamed from C311; DNP (none) -> x
- C212: renamed from C312; DNP (none) -> x
- C213: renamed from C313; DNP (none) -> x
- C214: renamed from C314; DNP (none) -> x
- C215: renamed from C315; DNP (none) -> x
- C216: renamed from C316; DNP (none) -> x
- C217: renamed from C317; DNP (none) -> x
- C218: renamed from C318; DNP (none) -> x
- C219: renamed from C319; DNP (none) -> x
- C220: renamed from C320; DNP (none) -> x
- C221: renamed from C321; DNP (none) -> x
- C222: renamed from C322; DNP (none) -> x
- C223: renamed from C323; DNP (none) -> x
- D201: renamed from D301; DNP (none) -> x
- D202: renamed from D302; DNP (none) -> x
- D203: renamed from D303; DNP (none) -> x
- D204: renamed from D304; DNP (none) -> x
- D205: renamed from D305; DNP (none) -> x
- L201: renamed from L301; DNP (none) -> x
- Q201: renamed from Q301; DNP (none) -> x
- Q202: renamed from Q302; DNP (none) -> x
- Q203: renamed from Q303; DNP (none) -> x
- R201: renamed from R301; DNP (none) -> x
- R202: renamed from R302; DNP (none) -> x
- R203: renamed from R303; DNP (none) -> x
- R204: renamed from R304; DNP (none) -> x
- R205: renamed from R305; DNP (none) -> x
- R206: renamed from R306; DNP (none) -> x
- R207: renamed from R307; DNP (none) -> x
- R208: renamed from R308; DNP (none) -> x
- R209: renamed from R309; DNP (none) -> x
- R210: renamed from R310; DNP (none) -> x
- R211: renamed from R311; DNP (none) -> x
- R212: renamed from R312; DNP (none) -> x
- R213: renamed from R313; DNP (none) -> x
- R214: renamed from R314; DNP (none) -> x
- R215: renamed from R315; DNP (none) -> x
- R216: renamed from R316; DNP (none) -> x
- R217: renamed from R317; DNP (none) -> x
- R218: renamed from R318; DNP (none) -> x
- R219: renamed from R319; DNP (none) -> x
- R220: renamed from R320; DNP (none) -> x
- R221: renamed from R321; DNP (none) -> x
- R222: renamed from R322; DNP (none) -> x
- R223: renamed from R323; DNP (none) -> x
- R224: renamed from R324; DNP (none) -> x
- R225: renamed from R325; DNP (none) -> x
- R226: renamed from R326; DNP (none) -> x
- U201: renamed from U301; DNP (none) -> x
- U202: renamed from U302; DNP (none) -> x
- U203: renamed from U303; DNP (none) -> x
- U204: renamed from U304; DNP (none) -> x
- U205: renamed from U305; DNP (none) -> x
- U206: renamed from U306; DNP (none) -> x
- U207: renamed from U307; DNP (none) -> x
- renumbered TP301 to TP201, TP302 to TP202, TP303 to TP203, TP304 to TP204, TP305 to TP205, TP306 to TP206, TP307 to TP207, TP308 to TP208, TP309 to TP209, TP310 to TP210, TP311 to TP211, TP312 to TP212, TP313 to TP213
