File: KiCAD_files/Microcontroller.kicad_sch (KiCad schematic)
At the start: 49 parts, among them J401 Conn_01x06_Male, J402 Conn_01x06_Male, J403 RJ45_LED_Shielded, J404 RJ45_LED_Shielded, P401 Power2, U401 OwnTech, U402 TCAN334GDR, U403 MCP1799T-5002H/TT, U404 AP1117-50

Commit message: WIP: added features for the RJ45 communication link. Added fast RS485 Added HRTIM Sync Added current share analog bus Added external VREF Added dedicated supply power supply pins for the data manager
Former-commit-id: 7d7dbd6688aaf47caa2ea5f91bf9cef552f6a24c
Parts:
- removed JP403, JP407: Jumper, Connector_PinHeader_2.54mm:PinHeader_1x02_P2.54mm_Vertical, symbol Jumper:Jumper_2_Open
- added C410: 100nF, Capacitor_SMD:C_1206_3216Metric, symbol Device:C_Small
- added C411, C412, C414, C416: 10pF, Capacitor_SMD:C_0805_2012Metric, symbol Device:C_Small
- added C413: 100nF, Capacitor_SMD:C_0805_2012Metric, symbol Device:C_Small
- added C415: 100nF, Footprints:C_0805_2012Metric, symbol Device:C_Small
- added D403: 1N4148WS, Diode_SMD:D_SOD-323, symbol Diode:1N4148WS
- added J405, J406: Conn_01x02_Male, Connector_JST:JST_EH_B2B-EH-A_1x02_P2.50mm_Vertical, symbol Connector:Conn_01x02_Male
- added JP403: Jumper, Connector_PinHeader_2.54mm:PinHeader_1x02_P2.54mm_Vertical, symbol Jumper:Jumper_2_Bridged
- added JP407, JP408, JP409: SolderJumper_2_Open, Jumper:SolderJumper-2_P1.3mm_Bridged_Pad1.0x1.5mm, symbol Jumper:SolderJumper_2_Bridged
- added JP410, JP416: Jumper_2_Bridged, Jumper:SolderJumper-2_P1.3mm_Open_Pad1.0x1.5mm, symbol Jumper:SolderJumper_2_Open
- added JP411, JP412, JP413, JP414, JP415: Jumper_2_Bridged, Jumper:SolderJumper-2_P1.3mm_Bridged_Pad1.0x1.5mm, symbol Jumper:SolderJumper_2_Bridged
- added R409, R411, R412, R413, R414, R415, R416, R417, R418, R419, R420, R421: 4.7k, Footprints:R_0805_2012Metric, symbol Device:R
- added R410: 120, Footprints:R_0805_2012Metric, symbol Device:R
- added R422: 47k, Footprints:R_0805_2012Metric, symbol Device:R
- added R423: 12k, Footprints:R_0805_2012Metric, symbol Device:R
- added R424: 1k, Footprints:R_0805_2012Metric, symbol Device:R_Small
- added TP409, TP410: TestPoint, Footprints:TestPoint_THTPad_D1.5mm_Drill0.7mm, symbol Connector:TestPoint
- added U405: LTC2850xS8, Package_SO:SOIC-8_3.9x4.9mm_P1.27mm, symbol Interface_UART:LTC2850xS8
- added U406: OPA2277, Package_SO:SOIC-8_3.9x4.9mm_P1.27mm, symbol Amplifier_Operational:OPA2277
- added U407: OPA316, Package_TO_SOT_SMD:SOT-353_SC-70-5, symbol Amplifier_Operational:TLV6001DCK
- TP401, TP402, TP403, TP404, TP405, TP406, TP407, TP408: footprint TestPoint:TestPoint_Pad_D1.0mm -> Footprints:TestPoint_THTPad_D1.5mm_Drill0.7mm
Connections:
- net +5VD: now also C410.1, R409.1, R421.1, R422.1, R424.1, U405.8 (VCC)
- net DAC2: now also R413.1, TP409.1
- net DGND: now also C410.2, C413.2, C414.1, C415.2, R411.2, R412.2, R414.1, R420.1, R423.2, TP410.1, U405.5 (GND), U406.4 (V-), U407.2 (V-)
- net PC13: now also JP412.2 (B)
- net USART1_{TX}: now also JP416.2 (B); no longer U401.23 (PB6)
- net VREF: now also JP407.2 (B)
- net SHARE-: now reaches J403.6
- net SHARE-: now also J404.6, R417.2, R418.2
- net GND_COM: now reaches J403.8
- net GND_COM: now also D402.2 (A), J404.8, R403.1, R405.1, J405.2 (Pin_2), J406.2 (Pin_2)
- net USART3_TX: now reaches U401.16 (PC10)
- net USART3_TX: now also U405.4 (DI)
- net USART3_RX: now reaches U401.17 (PC11)
- net USART3_RX: now also U405.1 (RO)
- net PC12: now reaches U401.19 (PC12)
- net PC12: now also JP413.2 (B)
- net ADC2_IN5: now reaches U401.41 (PC4)
- net ADC2_IN5: now also JP411.1 (A)
- net USART3_DE: now reaches U401.5 (PB14)
- net USART3_DE: now also R412.1, U405.2 (~{RE}), U405.3 (DE)
- net ADC4_IN5: now reaches U401.6 (PB15)
- net ADC4_IN5: now also JP406.1 (A), JP410.1 (A)
- net ADC3_IN1 renamed PB1
- net PB1: now also JP414.1 (A); no longer JP406.1 (A)
- removed net GND_CAN: D402.2 (A), J403.3, J403.7, J404.3, J404.7, R403.1, R405.1
- net PWR_CAN1 renamed PWR_COM1
- net PWR_COM1: now also J405.1 (Pin_1); no longer J403.4, J403.5
- net PWR_CAN2 renamed PWR_COM2
- net PWR_COM2: now also J406.1 (Pin_1); no longer J404.4, J404.5
- new net: C411.2, R415.2, R418.1, U406.6 (-)
- new net: C413.1, R421.2, U406.8 (V+)
- new net: C414.2, R422.2, R423.1, U407.1 (+)
- new net: JP409.2 (B), R411.1
- new net: C412.1, R414.2, R416.1, U406.2 (-)
- new net: JP408.1 (A), R409.2
- new net: C416.1, C416.2, JP407.1 (A), U407.3 (-), U407.4
- new net: D403.2 (A), U406.1
- new net: JP403.2 (B), R410.1
- new net: R419.1, U406.5 (+)
- new net: C411.1, JP410.2 (B), JP411.2 (B), R415.1, U406.7
- new net: C415.1, R424.2, U407.5 (V+)
- new net: R413.2, R417.1, U406.3 (+)
- new net A: J403.3, J404.3, JP403.1 (A), JP408.2 (B), U405.6 (A)
- new net B: J403.4, J404.4, JP409.1 (A), R410.2, U405.7 (B)
- new net HRTIM1_SCIN: J403.7, J404.7, JP414.2 (B), JP415.2 (B)
- new net PB6: JP415.1 (A), JP416.1 (A), U401.23 (PB6)
- new net SHARE+: C412.2, D403.1 (K), J403.5, J404.5, R416.2, R419.2, R420.2
- new net ~{STBY1}: JP413.1 (A), P401. (~{STBY2})
- new net ~{STBY2}: JP412.1 (A), P401. (~{STBY2})
- no-connect marks 17 -> 5
Other:
- note added: "Current sharing analog bus. Highest voltage is imposing its voltage to the bus"
- note added: "DAC2 can be used to provide a reference if this fails"
- note added: "Rudimentary 1.024V reference for measurement offset"
- note added: "Simulation available"
- note added: "https://tinyurl.com/2qg7lcok"
- note added: "https://tinyurl.com/mtt5xsmv"
- moved on the sheet: C401, C402, C403, C404, C405, C406, C407, C408, C409, D401, D402, F401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
