File: KiCAD_files/Microcontroller.kicad_sch (KiCad schematic)
At the start: 89 parts, among them J401 Conn_01x06_Male, J402 Conn_01x06_Male, J403 RJ45_LED_Shielded, J404 RJ45_LED_Shielded, J405 Conn_01x02_Male, J406 Conn_01x02_Male, P401 Power2, U401 OwnTech, U402 TCAN334GDR, U403 MCP1799T-5002H/TT, U404 AP1117-50, U405 LTC2850xS8, U406 OPA2277, U407 OPA316

Commit message: Feature Freeze PCB ordered
Former-commit-id: 656e77d39b103ec58b17965582500bfb0a5b80a0
Parts:
- removed J401, J402: Conn_01x06_Male, Connector_PinHeader_2.54mm:PinHeader_1x06_P2.54mm_Vertical, symbol Connector:Conn_01x06_Male
- removed JP402: SolderJumper_2_Open, Jumper:SolderJumper-2_P1.3mm_Bridged_Pad1.0x1.5mm, symbol Jumper:SolderJumper_2_Bridged
- removed JP416: Jumper_2_Bridged, Jumper:SolderJumper-2_P1.3mm_Open_Pad1.0x1.5mm, symbol Jumper:SolderJumper_2_Open
- added JP402: SolderJumper_2_Open, Jumper:SolderJumper-2_P1.3mm_Open_Pad1.0x1.5mm, symbol Jumper:SolderJumper_2_Open
- added JP417: Jumper_2_Bridged, Jumper:SolderJumper-2_P1.3mm_Bridged_Pad1.0x1.5mm, symbol Jumper:SolderJumper_2_Bridged
- added unit 3 of U401
- added unit 2 of U401
- U401: value OwnTech -> OwnTech_SPIN; footprint Footprints:OwnTech_MCU -> Footprints:OwnTech_SPINTHT; symbol Symbols:OwnTech_MCU -> Symbols:OwnTech_SPIN
Connections:
- net DAC2: now also JP402.1 (A), JP417.1 (A); no longer R413.1
- net VREF: now also JP402.2 (B)
- net DAC3_OUT1: now reaches U401.1 (PB11)
- net BOOT renamed FDCAN1_{RX}
- net SPI3_{MISO}: no longer names the net of U401.20 (PB4)
- net SPI3_{MOSI}: no longer names the net of U401.21 (PB5)
- net USART1_{RX}: no longer names the net of U401.24 (PB7)
- new net: JP417.2 (B), R413.1
- no-connect marks 5 -> 21
Other:
- note added: "Alternate 1.024V VREF signal from SoC integrated DAC2. Conflicts with Analog share bus"
- note removed: "1.024V VREF signal come from SoC integrated DAC2."
- note removed: "Standard headers for SPI and UART modules"
- note removed: "VREF2048 comes from the STM32G474 internal reference. It has to be configured through VREFBUF register."
- moved on the sheet: JP404, JP405, JP406, JP412, JP413, TP401, TP402, TP403, TP404, TP405, TP406, TP407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

Commit message: Added necessary information for BOM ordering
Former-commit-id: 116c703b052ef693f4f6c94bbef521d6efde9abc
Parts:
- C401: Manf# CC0805KRX7R9BB104 -> C0805C104K5RACTU
- C402, C403, C406, C407: #manf (none) -> 12105C106KAT2A; Manf# CL32B106KBJZW6E -> 12105C106KAT2A
- C404, C405, C408, C409: value 1µF -> 1uF; Manf# CL21B105KBFNFNE -> UMK212B7105KGHT
- C410: #manf (none) -> C1206C104K5RAC7867; Manf# CL32B106KBJZW6E -> C1206C104K5RAC7867
- C411, C412, C414, C416: value 10pF -> 20pF; footprint Capacitor_SMD:C_0805_2012Metric -> Footprints:C_0805_2012Metric; Manf# CL32B106KBJZW6E -> CC0805JRNPO9BN200
- C413: footprint Capacitor_SMD:C_0805_2012Metric -> Footprints:C_0805_2012Metric; Manf# CL32B106KBJZW6E -> C0805C104K5RACTU
- C415: Manf# (none) -> C0805C104K5RACTU
- D403: value 1N4148WS -> PMEG2010AEJ,115; footprint Diode_SMD:D_SOD-323 -> Footprints:D_SOD-323; Manf# (none) -> PMEG2010AEJ,115
- J405, J406: Manf# (none) -> B2B-EH-A(LF)(SN)
- JP401, JP403, JP404, JP405, JP406, JP410, JP411, JP412, JP413, JP414, JP415, JP417, P401, TH401, TH402, TP401, TP402, TP403, TP404, TP405, TP406, TP407, TP408, TP409, TP410, U401: DNP (none) -> x
- PS401: value MEE1S0505SC -> TEA 1-0505; Manf# (none) -> TEA 1-0505
- PS402: value MEE1S0512SC -> TBA 1-0512; Manf# (none) -> TBA 1-0512
- R401, R410: value 120 -> 120R
- R402, R404: value 330 -> 330R; Manf# CRCW0805330RFKEAC -> CR0805-FX-3300ELF
- R403, R405: value 3000 -> 3k
- R406, R407: Manf# PCF-W0805LF-03-2002-B-P-LT -> CR0805-FX-2002ELF
- R408: Manf# CR0805-FX-1200ELF -> CR0805-FX-1003ELF
- R409, R411, R412, R413, R414, R415, R416, R417, R418, R419, R420, R421: Manf# CR0805-FX-1200ELF -> CR0805-FX-4701ELF
- R422: Manf# CR0805-FX-1200ELF -> CR0805-FX-4702ELF
- R423: Manf# CR0805-FX-1200ELF -> CR0805-FX-1202ELF
- R424: Manf# (none) -> CR0805-FX-1001ELF
- U404: Manf# (none) -> AP1117-50
- U405: Manf# (none) -> LTC2850CS8#PBF
- U406: Manf# (none) -> MCP6487T-E/SN
- U407: Manf# (none) -> MCP6486UT-E/LT

Commit message: modified components references
Former-commit-id: 78eae5a79aa085afeb122b22fc422d089bf318c8
Parts:
- R408: Manf# CR0805-FX-1003ELF -> CR0805-J/-1R0ELF
Changed lines of the file:
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@@
       (effects (font (size 1.27 1.27)) hide)
     )
-    (property "Manf#" "CR0805-FX-1003ELF" (id 4) (at 269.24 198.755 0)
+    (property "Manf#" "CR0805-J/-1R0ELF" (id 4) (at 269.24 198.755 0)
       (effects (font (size 1.27 1.27)) hide)
     )

Commit message: Push up-to-date design files
Former-commit-id: f8cc17d9887a3e68c026953a0d17b74481171696
Parts:
- C401, C402, C403, C404, C405, C406, C407, C408, C409, C410, C411, C412, C413, C414, C415, C416, D401, D402, D403, F401, F402, J403, J404, J405, J406, PS401, PS402, R401, R402, R403, R404, R405, R406, R407, R408, R409, R410, R411, R412, R413, R414, R415, R416, R417, R418, R419, R420, R421, R422, R423, R424, U402, U403, U404, U405, U406, U407: DNP (none) -> x
