File: KiCAD_files/Power.kicad_sch (KiCad schematic)
At the start: 71 parts, among them J101 2604-1102, J102 2604-1102, J103 2604-1102, J104 2604-1102, J105 2604-1102, U101 AMC1311, U102 OPA316, U103 OPA316, U104 +-20A

Commit message: Feature Freeze PCB ordered
Former-commit-id: 656e77d39b103ec58b17965582500bfb0a5b80a0
Parts:
- added N101: Housing_Pad, Footprints:Guard_ring, symbol Mechanical:Housing_Pad
- H101, H102, H103, H104, H105, H106, H107, H108, H109: footprint MountingHole:MountingHole_2.7mm_M2.5 -> MountingHole:MountingHole_2.7mm_M2.5_DIN965_Pad_TopOnly; symbol Mechanical:MountingHole -> Mechanical:MountingHole_Pad
Connections:
- new net Earth_Protective: H101.1, H102.1, H103.1, H104.1, H105.1, H106.1, H107.1, H108.1, H109.1, N101.1 (PAD)

Commit message: Added necessary information for BOM ordering
Former-commit-id: 116c703b052ef693f4f6c94bbef521d6efde9abc
Parts:
- C101, C102, C124: #manf (none) -> C1206C104K5RAC7867; Manf# (none) -> C1206C104K5RAC7867
- C103, C117: Manf# (none) -> C0805C104K5RACTU
- C104, C105, C107, C108, C109, C110, C111, C112, C113, C114, C115, C116: Manf# (none) -> 12101C475K4T2A
- C106, C119: Manf# (none) -> CC0805JRNPO9BN200
- C118, C120, C121, C122: Manf# (none) -> ULT2C330MNL1GS
- C123: #manf (none) -> CL21C102JCFNNNE; Manf# (none) -> CL21C102JCFNNNE
- F101, F102, F103: Manf# (none) -> 0154008.DR
- H101, H102, H103, H104, H105, H106, H107, H108, H109, N101, TP101, TP102, TP103, TP104, TP105, TP106, TP107: DNP (none) -> x
- J101, J102, J103, J104, J105: Manf# (none) -> 2604-1102
- R101, R102, R106, R114, R119: Manf# (none) -> CR0805-FX-1001ELF
- R103, R104: Manf# (none) -> CR0805-FX-2702ELF
- R105, R107: Manf# (none) -> CR0805-FX-1202ELF
- R108, R109, R112, R113: Manf# (none) -> CR0805-FX-1004ELF
- R110, R116: Manf# (none) -> CR0805-FX-5901ELF
- R111, R115: Manf# (none) -> CR0805-FX-2002ELF
- R117: value 330K -> 330k; Manf# (none) -> CR0805-FX-3303ELF
- R118: value 5.6K -> 5.6k; Manf# (none) -> CR0805-FX-5601ELF
- U101: Manf# (none) -> AMC1311DWV
- U102, U103: Manf# (none) -> MCP6486UT-E/LT
- U104: Manf# (none) -> ACS723LLCTR-20AB
