File: KiCAD_files/microcontroller_mini.kicad_pcb (KiCad board)
At the start: 4 copper layers, 21 x 51 mm, 38 parts, among them J1 Conn_02x20_Top_Bottom, J101 Conn_01x05_Male, J102 Conn_01x06_Male, J2 USB_C_Receptacle_USB2.0, J8 FTSH-107-01-F-DV-K, SW1 KMR241NGLFS, SW2 KMR241NGLFS, U1 STM32G474RE, U3 WE-TVS-82400102, U4 AP1117-33, Y1 ECS-240-8-37-CKM-TR3 - 24MHz

Commit message: Feature Freeze PCB ordered
Former-commit-id: 656e77d39b103ec58b17965582500bfb0a5b80a0
Parts:
- removed the G*** at (111.5, 32.9)
- added G***: LOGO, Footprints:owntech_mini, F.Cu at (102.1, 86.3)
- added G***: LOGO, Footprints:owntech10mm, B.Cu at (96.0, 72.9)
- added kibuzzard-62C86036: G***, kibuzzard-62C86036, F.Cu at (91.6, 65.1)
- added kibuzzard-62C86188: G***, kibuzzard-62C86188, B.Cu at (95.6, 76.2)
- added kibuzzard-62C86242: G***, kibuzzard-62C86242, F.Cu at (92.0, 84.9)
- added kibuzzard-62C86250: G***, kibuzzard-62C86250, F.Cu at (92.0, 89.0)
- added kibuzzard-62C86302: G***, kibuzzard-62C86302, B.Cu at (101.9, 50.8)
- added kibuzzard-62C8630E: G***, kibuzzard-62C8630E, B.Cu at (101.5, 53.3)
- added kibuzzard-62C86317: G***, kibuzzard-62C86317, B.Cu at (92.3, 94.0)
- added kibuzzard-62C86317: G***, kibuzzard-62C86317, B.Cu at (92.3, 68.6)
- added kibuzzard-62C86317: G***, kibuzzard-62C86317, B.Cu at (101.9, 81.3)
- added kibuzzard-62C86317: G***, kibuzzard-62C86317, B.Cu at (101.9, 55.9)
- added kibuzzard-62C86317: G***, kibuzzard-62C86317, B.Cu at (101.9, 94.0)
- added kibuzzard-62C86317: G***, kibuzzard-62C86317, B.Cu at (89.5, 55.9)
- added kibuzzard-62C86317: G***, kibuzzard-62C86317, B.Cu at (101.9, 68.6)
- added kibuzzard-62C86317: G***, kibuzzard-62C86317, B.Cu at (92.3, 81.3)
- added kibuzzard-62C86324: G***, kibuzzard-62C86324, B.Cu at (102.3, 58.5)
- added kibuzzard-62C8632C: G***, kibuzzard-62C8632C, B.Cu at (101.5, 61.0)
- added kibuzzard-62C86335: G***, kibuzzard-62C86335, B.Cu at (102.3, 63.5)
- added kibuzzard-62C8633C: G***, kibuzzard-62C8633C, B.Cu at (102.3, 66.1)
- added kibuzzard-62C86349: G***, kibuzzard-62C86349, B.Cu at (102.3, 71.1)
- added kibuzzard-62C86353: G***, kibuzzard-62C86353, B.Cu at (102.3, 73.7)
- added kibuzzard-62C8635A: G***, kibuzzard-62C8635A, B.Cu at (102.3, 78.8)
- added kibuzzard-62C86362: G***, kibuzzard-62C86362, B.Cu at (102.3, 83.8)
- added kibuzzard-62C8636A: G***, kibuzzard-62C8636A, B.Cu at (102.3, 86.4)
- added kibuzzard-62C86371: G***, kibuzzard-62C86371, B.Cu at (102.3, 88.9)
- added kibuzzard-62C8637B: G***, kibuzzard-62C8637B, B.Cu at (102.3, 91.4)
- added kibuzzard-62C86384: G***, kibuzzard-62C86384, B.Cu at (101.9, 95.3)
- added kibuzzard-62C8639B: G***, kibuzzard-62C8639B, B.Cu at (89.4, 50.8)
- added kibuzzard-62C863A5: G***, kibuzzard-62C863A5, B.Cu at (89.4, 53.3)
- added kibuzzard-62C863AC: G***, kibuzzard-62C863AC, B.Cu at (92.3, 58.5)
- added kibuzzard-62C863B3: G***, kibuzzard-62C863B3, B.Cu at (95.9, 58.5)
- added kibuzzard-62C863BD: G***, kibuzzard-62C863BD, B.Cu at (92.3, 61.0)
- added kibuzzard-62C863C4: G***, kibuzzard-62C863C4, B.Cu at (95.6, 61.0)
- added kibuzzard-62C863D6: G***, kibuzzard-62C863D6, B.Cu at (92.3, 63.5)
- added kibuzzard-62C863DD: G***, kibuzzard-62C863DD, B.Cu at (95.6, 63.5)
- added kibuzzard-62C863E7: G***, kibuzzard-62C863E7, B.Cu at (91.9, 66.1)
- added kibuzzard-62C863ED: G***, kibuzzard-62C863ED, B.Cu at (95.6, 66.1)
- added kibuzzard-62C863F3: G***, kibuzzard-62C863F3, B.Cu at (95.6, 68.6)
- added kibuzzard-62C863FB: G***, kibuzzard-62C863FB, B.Cu at (89.1, 71.1)
- added kibuzzard-62C86401: G***, kibuzzard-62C86401, B.Cu at (89.1, 73.7)
- added kibuzzard-62C86407: G***, kibuzzard-62C86407, B.Cu at (89.1, 76.2)
- added kibuzzard-62C8640E: G***, kibuzzard-62C8640E, B.Cu at (89.1, 78.8)
- added kibuzzard-62C86415: G***, kibuzzard-62C86415, B.Cu at (96.0, 81.3)
- added kibuzzard-62C8641D: G***, kibuzzard-62C8641D, B.Cu at (96.0, 83.8)
- added kibuzzard-62C86424: G***, kibuzzard-62C86424, B.Cu at (96.0, 86.4)
- added kibuzzard-62C8642B: G***, kibuzzard-62C8642B, B.Cu at (95.6, 88.9)
- added kibuzzard-62C86431: G***, kibuzzard-62C86431, B.Cu at (95.6, 91.4)
- added kibuzzard-62C86437: G***, kibuzzard-62C86437, B.Cu at (95.6, 94.0)
- added kibuzzard-62C8643D: G***, kibuzzard-62C8643D, B.Cu at (95.6, 95.3)
- added kibuzzard-62C86450: G***, kibuzzard-62C86450, B.Cu at (91.9, 83.8)
- added kibuzzard-62C86458: G***, kibuzzard-62C86458, B.Cu at (92.3, 86.4)
- added kibuzzard-62C86461: G***, kibuzzard-62C86461, B.Cu at (92.3, 88.9)
- added kibuzzard-62C86468: G***, kibuzzard-62C86468, B.Cu at (92.3, 91.4)
- added kibuzzard-62C86470: G***, kibuzzard-62C86470, B.Cu at (92.3, 95.3)
- added kibuzzard-62C864F6: G***, kibuzzard-62C864F6, B.Cu at (102.3, 76.2)
- added kibuzzard-62C86A6F: G***, kibuzzard-62C86A6F, B.Cu at (87.7, 98.0)
- added kibuzzard-62C86A9B: G***, kibuzzard-62C86A9B, B.Cu at (90.4, 97.8)
- added kibuzzard-62C86AA4: G***, kibuzzard-62C86AA4, B.Cu at (99.4, 96.9)
- added kibuzzard-62C86AA4: G***, kibuzzard-62C86AA4, B.Cu at (91.9, 96.9)
- added kibuzzard-62C86AAB: G***, kibuzzard-62C86AAB, B.Cu at (94.6, 96.9)
- added kibuzzard-62C86AB2: G***, kibuzzard-62C86AB2, B.Cu at (96.8, 96.9)
- added kibuzzard-62C86ABB: G***, kibuzzard-62C86ABB, B.Cu at (101.4, 96.9)
- added kibuzzard-62C86AC0: G***, kibuzzard-62C86AC0, B.Cu at (103.3, 97.6)
- added kibuzzard-62C87078: G***, kibuzzard-62C87078, F.Cu at (95.7, 94.1)
- Y1: value ECS-240-8-37-CKM-TR3 - 24MHz -> 24MHz
- moved C9 0.32 mm to (102.9, 77.8)
Routing:
- net +3V3: track 94.5 -> 95.8 mm
- net PA0: track 4.35 -> 4.92 mm

Commit message: Added necessary information for BOM ordering
Former-commit-id: 116c703b052ef693f4f6c94bbef521d6efde9abc
Parts:
- U4: value AP1117-33 -> AZ1117-33
- Y1: value 24MHz -> ECS-240-8-37-CKM-TR3 - 24MHz
