File: KiCAD_files/Feeder.kicad_sch (KiCad schematic)
At the start: 59 parts, among them J505 Conn_01x03, Q501 60V N channel, Q502 TK13P25D,RQ, T501 PA2467NL, U501 NCP12700, U502 HMHA2801A, U503 TL431MFDT,215

Commit message: Added necessary information for BOM ordering
Former-commit-id: 116c703b052ef693f4f6c94bbef521d6efde9abc
Parts:
- C501, C502, C517, C518: #manf DNP -> (none); Manf# DNP -> 12101C475K4T2A
- C505: #manf CL21B102KBANNNC -> CL21C102JCFNNNE; Manf# CL21B102KBANNNC -> CL21C102JCFNNNE
- C507, C509: #manf CL21B105KBFNNNE -> UMK212B7105KGHT; Manf# CL21B105KBFNNNE -> UMK212B7105KGHT
- C515: #manf UMK325C7106KM-T -> 12105C106KAT2A; Manf# UMK325C7106KM-T -> 12105C106KAT2A
- C521: Manf# (none) -> EEE-FKE101XAP
- D507: Manf# STTH4R02U -> PU3DBH
- GND501, J505, JP501, VOUT_GND501: DNP (none) -> x
- L502: #manf (none) -> CBC3225T100M
- NTC501: value 100k -> 100kNTC
- R501: value 348K -> 348k
- R502: Manf# KTR10EZPF2702 -> CR0805-FX-2702ELF
- R504, R512, R514: value 1.4K -> 1.4k
- R505: value 2.2 -> 2.2R; Manf# RK73B2ATTDD2R2J -> CR0805AF/-2R20EAS
- R506: value 470 -> 470R; Manf# RC0805JR-07470RP -> CR0805-FX-4700ELF
- R507, R511, R516: value 10 -> 10R; Manf# CRCW080510R0JNEAC -> CR0805-FX-10R0ELF
- R518: Manf# RC0805FR-0714K7L -> CR0805-FX-2702ELF
- U502: #manf HMHA2801A -> HMHA2801A; Manf# HMHA2801A -> HMHA2801A

Commit message: modified components references
Former-commit-id: 78eae5a79aa085afeb122b22fc422d089bf318c8
Parts:
- C519, C520: Manf# DNP -> GRM21BR72A474KA73L
- R503: Manf# KTR10EZPJ104 -> CR0805-FX-1003ELF
- U502: Manf# HMHA2801A -> FODM217A
Changed lines of the file:
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@@
       (effects (font (size 1.27 1.27)) hide)
     )
-    (property "Manf#" "KTR10EZPJ104" (id 5) (at 114.3 139.7 0)
+    (property "Manf#" "CR0805-FX-1003ELF" (id 5) (at 114.3 139.7 0)
       (effects (font (size 1.27 1.27)) hide)
     )
@@
       (effects (font (size 1.27 1.27)) (justify left) hide)
     )
-    (property "Manf#" "HMHA2801A" (id 4) (at 229.87 174.625 0)
+    (property "Manf#" "FODM217A" (id 4) (at 229.87 174.625 0)
       (effects (font (size 1.27 1.27)) hide)
     )
@@
       (effects (font (size 1.27 1.27)) hide)
     )
-    (property "Manf#" "DNP" (id 5) (at 35.56 64.135 0)
+    (property "Manf#" "GRM21BR72A474KA73L" (id 5) (at 35.56 64.135 0)
       (effects (font (size 1.27 1.27)) hide)
     )
@@
       (effects (font (size 1.27 1.27)) hide)
     )
-    (property "Manf#" "DNP" (id 5) (at 35.56 80.645 0)
-      (effects (font (size 1.27 1.27)) hide)
-    )
+    (property "Manf#" "GRM21BR72A474KA73L" (id 5) (at 35.56 80.645 0)
+      (effects (font (size 1.27 1.27)) hide)
+    )

Commit message: Push up-to-date design files
Former-commit-id: f8cc17d9887a3e68c026953a0d17b74481171696
Parts:
- J505: DNP x -> (none)
Changed lines of the file:
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@@
       (effects (font (size 1.27 1.27)) hide)
     )
-    (property "DNP" "x" (id 4) (at 327.025 93.345 0)
+    (property "DNP" "" (id 4) (at 327.025 93.345 0)
       (effects (font (size 1.27 1.27)) hide)
     )
